Commit message: description

File: tocabi_description/robots/dyros_tocabi.urdf (robot description, URDF)
Before this commit: robot dyros_red_description, 34 links, 33 joints
Links:
- link Head_Link: geometry collision cylinder length=0.043 radius=0.07; visual mesh filename=package://tocabi_description/meshes/head.STL
- link L_AnkleCenter_Link: geometry collision box size=0.1045 0.06 0.095; visual mesh filename=package://tocabi_description/meshes/AnkleCenter_L_Link.STL
- link L_AnkleRoll_Link: geometry collision box size=0.26 0.1 0.027; collision cylinder length=0.0625 radius=0.045
- link L_Armlink_Link: geometry collision cylinder length=0.16 radius=0.04; visual mesh filename=package://tocabi_description/meshes/L_arm.STL
- link L_Elbow_Link: geometry collision cylinder length=0.08 radius=0.04; collision cylinder length=0.08 radius=0.04
- link L_Forearm_Link: geometry collision cylinder length=0.08 radius=0.025; collision cylinder length=0.1 radius=0.04
- link L_HipCenter_Link: geometry collision box size=0.1045 0.06 0.095; visual mesh filename=package://tocabi_description/meshes/HipCenter_L_Link.STL
- link L_HipRoll_Link: geometry collision box size=0.012 0.072 0.095; collision box size=0.012 0.072 0.095
- link L_Knee_Link: geometry collision cylinder length=0.200 radius=0.06; visual mesh filename=package://tocabi_description/meshes/Knee_L_Link.STL
- link L_Shoulder1_Link: geometry collision cylinder length=0.11 radius=0.04; visual mesh filename=package://tocabi_description/meshes/L_shoulder1.STL
- link L_Shoulder2_Link: geometry collision cylinder length=0.05 radius=0.04; visual mesh filename=package://tocabi_description/meshes/L_shoulder2.STL
- link L_Shoulder3_Link: geometry collision cylinder length=0.12 radius=0.04; visual mesh filename=package://tocabi_description/meshes/L_shoulder3.STL
- link L_Thigh_Link: geometry collision cylinder length=0.07763 radius=0.049; collision cylinder length=0.2175 radius=0.06
- link L_Wrist1_Link: geometry collision cylinder length=0.06 radius=0.02; visual mesh filename=package://tocabi_description/meshes/L_wrist1.STL
- link Neck_Link: geometry collision cylinder length=0.043 radius=0.07; visual mesh filename=package://tocabi_description/meshes/neck.STL
- link Pelvis_Link: geometry collision box size=0.141 0.305 0.05; collision cylinder length=0.088 radius=0.045
- link R_AnkleCenter_Link: geometry collision box size=0.1045 0.06 0.095; visual mesh filename=package://tocabi_description/meshes/AnkleCenter_R_Link.STL
- link R_AnkleRoll_Link: geometry collision box size=0.26 0.1 0.027; collision cylinder length=0.0625 radius=0.045
- link R_Armlink_Link: geometry collision cylinder length=0.16 radius=0.04; visual mesh filename=package://tocabi_description/meshes/R_arm.STL
- link R_Elbow_Link: geometry collision cylinder length=0.08 radius=0.04; collision cylinder length=0.08 radius=0.04
- link R_Forearm_Link: geometry collision cylinder length=0.08 radius=0.025; collision cylinder length=0.1 radius=0.04
- link R_HipCenter_Link: geometry collision box size=0.1045 0.06 0.095; visual mesh filename=package://tocabi_description/meshes/HipCenter_R_Link.STL
- link R_HipRoll_Link: geometry collision box size=0.012 0.072 0.095; collision box size=0.012 0.072 0.095
- link R_Knee_Link: geometry collision cylinder length=0.200 radius=0.06; visual mesh filename=package://tocabi_description/meshes/Knee_R_Link.STL
- link R_Shoulder1_Link: geometry collision cylinder length=0.11 radius=0.04; visual mesh filename=package://tocabi_description/meshes/R_shoulder1.STL
- link R_Shoulder2_Link: geometry collision cylinder length=0.05 radius=0.04; visual mesh filename=package://tocabi_description/meshes/R_shoulder2.STL
- link R_Shoulder3_Link: geometry collision cylinder length=0.12 radius=0.04; visual mesh filename=package://tocabi_description/meshes/R_shoulder3.STL
- link R_Thigh_Link: geometry collision cylinder length=0.07763 radius=0.049; collision cylinder length=0.2175 radius=0.06
- link R_Wrist1_Link: geometry collision cylinder length=0.06 radius=0.02; visual mesh filename=package://tocabi_description/meshes/R_wrist1.STL
- link Upperbody_Link: geometry collision box size=0.12 0.07 0.14; collision box size=0.21 0.11 0.07
- link Waist1_Link: geometry collision box size=0.094 0.01 0.091; collision box size=0.094 0.01 0.091
- link Waist2_Link: geometry collision box size=0.09 0.1 0.091; collision box size=0.1 0.1 0.06

Commit message: urdf & code revise

File: tocabi_description/robots/dyros_tocabi.urdf (robot description, URDF)
Before this commit: robot dyros_tocabi, 34 links, 33 joints
Joints:
- joint Head_Joint: limit lower=1.54 upper=1.54 effort=500 velocity=100 -> lower=-1.54 upper=1.54 effort=500 velocity=100; origin xyz=0.0 0.0 0.0275 rpy=0 0 -1.54 -> xyz=0.0 0.0 0.0275 rpy=0 0 0
- joint Neck_Joint: limit lower=1.54 upper=1.54 effort=500 velocity=100 -> lower=-1.54 upper=1.54 effort=500 velocity=100

Commit message: revise xml,urdf, cnt2nm

File: tocabi_description/robots/dyros_tocabi.urdf (robot description, URDF)
Before this commit: robot dyros_tocabi, 34 links, 33 joints
Links:
- link L_AnkleRoll_Link: mass 3.464 -> 3.590; geometry collision box size=0.3 0.17 0.027; collision cylinder length=0.0625 radius=0.045
- link L_Wrist2_Link: mass 1 -> 0.001
- link Pelvis_Link: mass 0.90054 -> 12.19525
- link R_AnkleRoll_Link: mass 3.464 -> 3.590; geometry collision box size=0.3 0.17 0.027; collision cylinder length=0.0625 radius=0.045
- link R_Wrist2_Link: mass 1 -> 0.001
- link Upperbody_Link: mass 16.43395 -> 16.43384
- link Waist1_Link: mass 0.74235 -> 0.89722
- link Waist2_Link: mass 3.27104 -> 3.752
Joints:
- joint R_AnkleRoll_Joint: origin xyz=0 0 0 rpy=2.77555756156282E-17 1.48042453629419E-16 -5.37756273475549E-16 -> xyz=0 0 0 rpy=0 0 0
- joint Waist1_Joint: origin xyz=0 0 0.18 rpy=0 0 0 -> xyz=0 0 0.1779 rpy=0 0 0

Commit message: xml revise

File: tocabi_description/robots/dyros_tocabi.urdf (robot description, URDF)
Before this commit: robot dyros_tocabi_description, 34 links, 33 joints
Links:
- added link L_Foot_Link, mass 2.326; collision box size=0.3 0.17 0.027; collision cylinder length=0.0625 radius=0.045
- added link R_Foot_Link, mass 2.326; collision box size=0.3 0.17 0.027; collision cylinder length=0.0625 radius=0.045
- link L_AnkleRoll_Link: mass 3.590 -> 1.26426; geometry collision cylinder length=0.0625 radius=0.045; visual mesh filename=package://tocabi_description/meshes/AnkleRoll_L_Link.STL
- link R_AnkleRoll_Link: mass 3.590 -> 1.26426; geometry collision cylinder length=0.0625 radius=0.045; visual mesh filename=package://tocabi_description/meshes/AnkleRoll_R_Link.STL
Joints:
- added joint L_Foot_Joint: type fixed, parent L_AnkleRoll_Link, child L_Foot_Link, origin xyz=0 0 0 rpy=0 0 0, axis 0 0 0, limit lower=-3.14 upper=3.14 effort=500 velocity=100
- added joint R_Foot_Joint: type fixed, parent R_AnkleRoll_Link, child R_Foot_Link, origin xyz=0 0 0 rpy=0 0 0, axis 0 0 0, limit lower=-3.14 upper=3.14 effort=500 velocity=100

Commit message: jointalign

File: tocabi_description/robots/dyros_tocabi.urdf (robot description, URDF)
Before this commit: robot dyros_tocabi_description, 36 links, 35 joints
Joints:
- removed joint L_AnkleCenter_Joint
- removed joint L_HipCenter_Joint
- removed joint L_Thigh_Joint
- removed joint R_AnkleCenter_Joint
- removed joint R_HipCenter_Joint
- removed joint R_Thigh_Joint
- added joint L_AnklePitch_Joint: type revolute, parent L_Knee_Link, child L_AnkleCenter_Link, origin xyz=0 0 -0.350000000051828 rpy=2.57102424745274E-31 -1.5978825624527E-16 1.89651504296143E-16, axis 0 1 0, limit lower=-3.14 upper=3.14 effort=500 velocity=100
- added joint L_HipPitch_Joint: type revolute, parent L_HipCenter_Link, child L_Thigh_Link, origin xyz=0 0 0 rpy=-2.77555756156289E-17 -1.88969769143558E-16 -1.36928250674653E-16, axis 0 1 0, limit lower=-3.14 upper=3.14 effort=500 velocity=100
- added joint L_HipYaw_Joint: type revolute, parent Pelvis_Link, child L_HipRoll_Link, origin xyz=0 0.1025 -0.1225 rpy=0 0 0, axis 0 0 1, limit lower=-3.14 upper=3.14 effort=500 velocity=100
- added joint R_AnklePitch_Joint: type revolute, parent R_Knee_Link, child R_AnkleCenter_Link, origin xyz=0 0 -0.35 rpy=-2.77555756156282E-17 -1.48042453629419E-16 5.37756273475549E-16, axis 0 1 0, limit lower=-3.14 upper=3.14 effort=500 velocity=100
- added joint R_HipPitch_Joint: type revolute, parent R_HipCenter_Link, child R_Thigh_Link, origin xyz=0 0 0 rpy=-1.38777878078143E-17 -2.74984739744835E-16 -4.49346870585602E-16, axis 0 1 0, limit lower=-3.14 upper=3.14 effort=500 velocity=100
- added joint R_HipYaw_Joint: type revolute, parent Pelvis_Link, child R_HipRoll_Link, origin xyz=0 -0.1025 -0.1225 rpy=0 0 0, axis 0 0 1, limit lower=-3.14 upper=3.14 effort=500 velocity=100
- joint L_HipRoll_Joint: axis 0 0 1 -> 1 0 0; child L_HipRoll_Link -> L_HipCenter_Link; origin xyz=0 0.1025 -0.1225 rpy=0 0 0 -> xyz=0 0 0 rpy=2.77555756156289E-17 1.88969769143558E-16 1.36928250674653E-16; parent Pelvis_Link -> L_HipRoll_Link
- joint R_HipRoll_Joint: axis 0 0 1 -> 1 0 0; child R_HipRoll_Link -> R_HipCenter_Link; origin xyz=0 -0.1025 -0.1225 rpy=0 0 0 -> xyz=0 0 0 rpy=1.38777878078145E-17 2.74984739744835E-16 4.49346870585602E-16; parent Pelvis_Link -> R_HipRoll_Link

Commit message: add customcontroller

File: tocabi_description/robots/dyros_tocabi.urdf (robot description, URDF)
Before this commit: robot dyros_tocabi_description, 36 links, 35 joints
Links:
- link Upperbody_Link: mass 16.43384 -> 16.93384

Commit message: tune urdf

File: tocabi_description/robots/dyros_tocabi.urdf (robot description, URDF)
Before this commit: robot dyros_tocabi_description, 36 links, 35 joints
Links:
- link Head_Link: mass 3.46332 -> 0.006332
- link L_Armlink_Link: mass 0.43517 -> 0.58517
- link L_Elbow_Link: mass 1.96511 -> 2.06511
- link L_Forearm_Link: mass 0.30234 -> 0.35234
- link R_Armlink_Link: mass 0.43517 -> 0.58517
- link R_Elbow_Link: mass 1.96511 -> 2.06511
- link R_Forearm_Link: mass 0.30234 -> 0.35234

Commit message: commit

File: tocabi_description/robots/dyros_tocabi.urdf (robot description, URDF)
Before this commit: robot dyros_tocabi_description, 36 links, 35 joints
Links:
- link L_AnkleRoll_Link: mass 1.26426 -> 2.16426
- link R_AnkleRoll_Link: mass 1.26426 -> 2.16426

Commit message: Tune urdf

File: tocabi_description/robots/dyros_tocabi.urdf (robot description, URDF)
Before this commit: robot dyros_tocabi_description, 36 links, 35 joints
Links:
- link L_AnkleRoll_Link: mass 2.16426 -> 1.76426
- link R_AnkleRoll_Link: mass 2.16426 -> 1.76426
- link Upperbody_Link: mass 16.93384 -> 18.13384

Commit message: edit model files

File: tocabi_description/robots/dyros_tocabi.urdf (robot description, URDF)
Before this commit: robot dyros_tocabi_description, 36 links, 35 joints
Links:
- link L_Wrist2_Link: geometry collision box size=0.06 0.02 0.06; visual box size=0.06 0.02 0.06
- link R_Wrist2_Link: geometry collision box size=0.06 0.02 0.06; visual box size=0.06 0.02 0.06

Commit message: Fixx 4contact

File: tocabi_description/robots/dyros_tocabi.urdf (robot description, URDF)
Before this commit: robot dyros_tocabi_description, 36 links, 35 joints
Links:
- link L_Wrist2_Link: mass 0.001 -> 0.1; geometry collision box size=0.06 0.06 0.02; visual box size=0.06 0.06 0.02
- link R_Wrist2_Link: mass 0.001 -> 0.1; geometry collision box size=0.06 0.06 0.02; visual box size=0.06 0.06 0.02
Joints:
- joint L_Wrist2_Joint: origin xyz=0 0.046 0 rpy=0 0 0 -> xyz=0 0.046 0 rpy=1.5708 3.1415 0
- joint R_Wrist2_Joint: origin xyz=0 -0.046 0 rpy=0 0 0 -> xyz=0 -0.046 0 rpy=-1.5708 3.1415 0

Commit message: Move origin of model file

File: tocabi_description/robots/dyros_tocabi.urdf (robot description, URDF)
Before this commit: robot dyros_tocabi_description, 36 links, 35 joints
Joints:
- joint L_HipYaw_Joint: origin xyz=0 0.1025 -0.1225 rpy=0 0 0 -> xyz=0.11 0.1025 -0.1025 rpy=0 0 0
- joint R_HipYaw_Joint: origin xyz=0 -0.1025 -0.1225 rpy=0 0 0 -> xyz=0.11 -0.1025 -0.1025 rpy=0 0 0
- joint Waist1_Joint: origin xyz=0 0 0.1779 rpy=0 0 0 -> xyz=0.11 0 0.1979 rpy=0 0 0

Commit message: model_fix

File: tocabi_description/robots/dyros_tocabi.urdf (robot description, URDF)
Before this commit: robot dyros_tocabi_description, 36 links, 35 joints
Joints:
- joint L_Wrist2_Joint: axis 0 0 1 -> 0 1 0
- joint R_Wrist2_Joint: axis 0 0 1 -> 0 -1 0

Commit message: qp3

File: tocabi_description/robots/dyros_tocabi.urdf (robot description, URDF)
Before this commit: robot dyros_tocabi_description, 36 links, 35 joints
Links:
- link L_AnkleRoll_Link: mass 1.76426 -> 1.26426
- link R_AnkleRoll_Link: mass 1.76426 -> 1.26426
