Commit message: after avatar exp editted qb allegro urdf

File: tocabi_description/robots/dyros_tocabi_with_allegro_qb.urdf (robot description, URDF)
Before this commit: robot dyros_tocabi_description, 36 links, 35 joints
Links:
- link L_Wrist2_Link: mass 1.070 -> 0.6
- link R_Wrist2_Link: mass 1.7 -> 1.4
